File: Projetos Eagle/BUZZER.sch (EAGLE design)
At the start: 7 parts, among them J1 CONECTOR_IN, J2 CONECTOR, Q1 BC817, U1 74HC132

Commit message: correção de pads e adição de label para versionamento
Parts:
- J1: value CONECTOR_IN -> CONECTOR_MACHO; device Eletroblocks Lib:CONECTOR_IN -> Eletroblocks Lib:CONECTOR_MACHO
- J2: value CONECTOR -> CONECTOR_FEMEA; device Eletroblocks Lib:CONECTOR -> Eletroblocks Lib:CONECTOR_FEMEA
Changed lines of the file:
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@@
 <part name="P+4" library="supply1" library_urn="urn:adsk.eagle:library:371" deviceset="VCC" device=""/>
 <part name="GND2" library="supply1" library_urn="urn:adsk.eagle:library:371" deviceset="GND" device=""/>
-<part name="J1" library="Eletroblocks Lib" deviceset="CONECTOR_IN" device="" override_package3d_urn="urn:adsk.eagle:package:22321382/3" override_package_urn="urn:adsk.eagle:footprint:22321383/1"/>
-<part name="J2" library="Eletroblocks Lib" deviceset="CONECTOR" device="" override_package3d_urn="urn:adsk.eagle:package:22308003/4" override_package_urn="urn:adsk.eagle:footprint:22308004/1"/>
+<part name="J1" library="Eletroblocks Lib" deviceset="CONECTOR_MACHO" device="" override_package3d_urn="urn:adsk.eagle:package:22321382/3" override_package_urn="urn:adsk.eagle:footprint:22321383/1" override_locally_modified="yes"/>
+<part name="J2" library="Eletroblocks Lib" deviceset="CONECTOR_FEMEA" device="" override_package3d_urn="urn:adsk.eagle:package:22308003/4" override_package_urn="urn:adsk.eagle:footprint:22308004/1" override_locally_modified="yes"/>
 <part name="P+1" library="supply1" library_urn="urn:adsk.eagle:library:371" deviceset="VCC" device=""/>
 <part name="GND4" library="supply1" library_urn="urn:adsk.eagle:library:371" deviceset="GND" device=""/>
